Commit message: add hydrus new model for checking ceiling effect

File: robots/hydrus/urdf/common.xacro (robot description, xacro)
@@ -6,5 +6,7 @@
   <thrust_link name="thrust" />
   <!-- kinematics [m] -->
-  <xacro:property name="link_length" value=".6" />
+  <xacro:property name="link_length" value=".580" />
+  <xacro:property name="link_length_2" value=".575" />
+  <xacro:property name="link_length_3" value=".625" />
   <xacro:property name="protector_radius" value=".1925" />
   <xacro:property name="head_leg_offset" value="${0.3 - 0.25884}" />
@@ -20,5 +22,5 @@
   <xacro:property name="max_force" value="20.0" /> <!-- [N] -->
   <xacro:property name="min_force" value="1.0" /> <!-- [N] -->
-  <xacro:macro name="link_model" params="type with_leg:=${with_leg} old_version:=${old_version} tilt_mode:=${tilt_mode} tilt_angle:=${tilt_angle} prop_15inch:=${prop_15inch}">
+  <xacro:macro name="link_model" params="type with_leg:=${with_leg} old_version:=${old_version} tilt_mode:=${tilt_mode} tilt_angle:=${tilt_angle} prop_15inch:=${prop_15inch} mesh_ext:=dae support_ce:=${support_ce}">
     <!-- for fcl in planning -->
     <collision>
@@ -37,14 +39,17 @@
     </collision>
     <visual>
+      <!-- old version -->
       <xacro:if value="${old_version == 1}">
         <origin rpy="0 0 0" xyz="${link_length* 0.5} 0 0"/>
         <geometry>
-          <mesh filename="package://hydrus/urdf/mesh/ver1/link/${type}_link.dae"/>
+          <mesh filename="package://hydrus/urdf/mesh/ver1/link/${type}_link.${mesh_ext}"/>
         </geometry>
       </xacro:if>
+      <!-- new version -->
       <xacro:unless value="${old_version == 1}">
-        <origin rpy="0 0 0" xyz="${link_length* 0.5} 0 0"/>
-        <geometry>
-          <xacro:if value="${tilt_mode == 1}">
+        <!-- tilt model -->
+        <xacro:if value="${tilt_mode == 1}">
+          <origin rpy="0 0 0" xyz="${link_length* 0.5} 0 0"/>
+          <geometry>
             <xacro:if value="${prop_15inch == 1}">
               <mesh filename="package://hydrus/urdf/mesh/ver2/link/tilt_${tilt_angle}deg_15inch_link${type}.dae"/>
@@ -53,9 +58,25 @@
               <mesh filename="package://hydrus/urdf/mesh/ver2/link/tilt_${tilt_angle}deg_link${type}.dae"/>
             </xacro:unless>
+          </geometry>
+        </xacro:if>
+        <!-- non-tilt CE/ver3 model -->
+        <xacro:unless value="${tilt_mode == 1}">
+          <xacro:if value="${type == 1}">
+            <!-- <origin rpy="0 0 0" xyz="0.020 0.000 0.000"/> -->
+            <origin rpy="0 0 0" xyz="0.000 0.000 0.000"/>
           </xacro:if>
-          <xacro:unless value="${tilt_mode == 1}">
-            <mesh filename="package://hydrus/urdf/mesh/ver2/link/link${type}.dae"/>
-          </xacro:unless>
-        </geometry>
+          <xacro:if value="${type == 2}">
+            <origin rpy="0 0 0" xyz="0.000 0.000 0.000"/>
+          </xacro:if>
+          <xacro:if value="${type == 3}">
+            <origin rpy="0 0 0" xyz="0.000 0.000 0.000"/>
+          </xacro:if>
+          <xacro:if value="${type == 4}">
+            <origin rpy="0 0 0" xyz="0.000 -0.000 0.000"/>
+          </xacro:if>
+          <geometry>
+            <mesh filename="package://hydrus/urdf/mesh/ver3/link/link${type}.${mesh_ext}"/>
+          </geometry>
+        </xacro:unless>
       </xacro:unless>
     </visual>
@@ -126,4 +147,18 @@
     </xacro:extra_module>
   </xacro:macro>
+  <!-- support_ce -->
+  <xacro:macro name="support_ce_module" params="name parent *origin">
+    <xacro:extra_module name="${name}" parent="${parent}" visible="1"
+                        model_url="package://hydrus/urdf/mesh/ver3/support_ce/support_ce.${mesh_ext}">
+      <xacro:insert_block name="origin"/>
+      <inertial>
+        <origin xyz="0 0 0" rpy="0 0 0"/>
+        <mass value="0.001"/>
+        <inertia ixx="0.000001" ixy="0.0" ixz="0.0"
+                iyy="0.000001" iyz="0.0"
+                izz="0.000001"/>
+      </inertial>
+    </xacro:extra_module>
+  </xacro:macro>
   <!-- friction -->
   <xacro:macro name="friction" params="self">

File: robots/hydrus/urdf/link.urdf.xacro (robot description, xacro)
@@ -3,5 +3,5 @@
     xmlns:xacro="http://www.ros.org/wiki/xacro" name="hydrus_link" >
   <!-- D-H kai description(different from prof.nakamura) -->
-  <xacro:macro name="hydrus_link" params="links self rotor_direction with_leg:=1 with_battery:=1 old_version:=0 tilt_mode:=0 tilt_angle:=0 prop_15inch:=0">
+  <xacro:macro name="hydrus_link" params="links self rotor_direction with_leg:=1 with_battery:=1 old_version:=0 tilt_mode:=0 tilt_angle:=0 prop_15inch:=0 mesh_ext:=dae support_ce:=0">
     <xacro:if value="${old_version == 1}">
       <!-- link -->
@@ -16,5 +16,5 @@
                 ixy="0.000021" ixz="0.000372" iyz="0.000000"/>
           </inertial>
-          <xacro:link_model type="head" />
+          <xacro:link_model type="head" mesh_ext="${mesh_ext}" />
         </xacro:if>
         <xacro:unless value="${self == 1}">
@@ -28,5 +28,5 @@
                   ixy="0.000020" ixz="-0.000076" iyz="0.000000"/>
             </inertial>
-            <xacro:link_model type="end" />
+            <xacro:link_model type="end" mesh_ext="${mesh_ext}" />
           </xacro:if>
           <xacro:unless value="${self == links}">
@@ -39,5 +39,5 @@
                   ixy="0.000021" ixz="0.000260" iyz="0.000000"/>
             </inertial>
-            <xacro:link_model type="general" />
+            <xacro:link_model type="general" mesh_ext="${mesh_ext}" />
           </xacro:unless>
         </xacro:unless>
@@ -78,5 +78,5 @@
             </inertial>
           </xacro:unless>
-          <xacro:link_model type="1" />
+          <xacro:link_model type="1" mesh_ext="${mesh_ext}" />
         </xacro:if>
         <xacro:unless value="${self == 1}">
@@ -108,9 +108,9 @@
                 <mass value="0.590"/> <!-- +DCDC -->
                 <inertia
-                    ixx="0.00179" iyy="0.01581" izz="0.01692"
-                    ixy="0.00000" ixz="-0.00067" iyz="0.00000"/>
+                    ixx="0.00040638959" ixy="0.00000778848" ixz="-0.00096295536"
+                    iyy="0.01635382606" iyz="-0.00000232615" izz="0.01606515391"/>
               </inertial>
             </xacro:unless>
-            <xacro:link_model type="4" />
+            <xacro:link_model type="4" mesh_ext="${mesh_ext}" />
           </xacro:if>
           <xacro:unless value="${self == links}">
@@ -139,12 +139,12 @@
               <xacro:unless value="${tilt_mode == 1}">
                 <inertial>
-                  <origin xyz="${link_length * 0.5} 0.0 0.01287" rpy="0 0 0"/>
+                  <origin xyz="0.32860 0.00000 0.01523" rpy="0 0 0"/>
                   <mass value="0.55744"/>
                   <inertia
-                      ixx="0.00171" iyy="0.01727" izz="0.01844"
-                      ixy="0.00000" ixz="0.00001" iyz="0.00000"/>
+                      ixx="0.00038023587" ixy="0.00000386183" ixz="0.00082294684"
+                      iyy="0.01861673811" iyz="0.00000214317" izz="0.01835189951"/>
                 </inertial>
               </xacro:unless>
-              <xacro:link_model type="2" />
+              <xacro:link_model type="2" mesh_ext="${mesh_ext}" />
             </xacro:if>
             <!-- general -->
@@ -172,12 +172,12 @@
               <xacro:unless value="${tilt_mode == 1}">
                 <inertial>
-                  <origin xyz="${link_length * 0.5 - 0.0317} 0.0 0.01836" rpy="0 0 0"/>
+                  <origin xyz="0.31840 -0.00006 0.00765" rpy="0 0 0"/>
                   <mass value="0.63453"/>
                   <inertia
-                      ixx="0.00182" iyy="0.02232" izz="0.02254"
-                      ixy="0.00000" ixz="-0.00077" iyz="0.00000"/>
+                      ixx="0.00029131008" ixy="-0.00000514804" ixz="0.00001047486"
+                      iyy="0.02355504631" iyz="0.00000120004" izz="0.02339409703"/>
                 </inertial>
               </xacro:unless>
-              <xacro:link_model type="3" />
+              <xacro:link_model type="3" mesh_ext="${mesh_ext}"/>
             </xacro:unless>
           </xacro:unless>
@@ -200,5 +200,16 @@
       </xacro:if>
       <xacro:unless value="${tilt_mode == 1}">
-        <origin rpy="0 0 0" xyz="${link_length* 0.5} 0 0.013"/>
+        <xacro:if value="${self == 1}">
+          <origin rpy="0 0 0" xyz="${link_length*0.5-0.010} 0.000 0.013"/>
+        </xacro:if>
+        <xacro:if value="${self == 2}">
+          <origin rpy="0 0 0" xyz="${link_length_2*0.5+0.0125} 0.000 0.013"/>
+        </xacro:if>
+        <xacro:if value="${self == 3}">
+          <origin rpy="0 0 0" xyz="${link_length_3*0.5+0.01375} 0.000 0.013"/>
+        </xacro:if>
+        <xacro:if value="${self == 4}">
+          <origin rpy="0 0 0" xyz="${link_length_2*0.5+0.01375} 0.000 0.013"/>
+        </xacro:if>
       </xacro:unless>
       <axis xyz="0 0 ${rotor_direction}"/>
@@ -249,4 +260,31 @@
       </xacro:extra_module>
     </xacro:if>
+    <!-- support_ce module -->
+    <xacro:if value="${support_ce == 1}">
+      <!-- support_ce1: link1 -->
+      <xacro:if value="${self == 1}">
+        <xacro:support_ce_module name="support_ce1" parent="link1">
+          <origin xyz="${head_leg_offset} 0.0 0.01" rpy="0 0 0"/>
+        </xacro:support_ce_module>
+      </xacro:if>
+      <!-- support_ce2: link2 -->
+      <xacro:if value="${self == 2}">
+        <xacro:support_ce_module name="support_ce2" parent="link2">
+          <origin xyz="0.05 0.000 0.01" rpy="0 0 0"/>
+        </xacro:support_ce_module>
+      </xacro:if>
+      <!-- support_ce3: link3 -->
+      <xacro:if value="${self == 3}">
+        <xacro:support_ce_module name="support_ce3" parent="link3">
+          <origin xyz="${link_length_3-0.05} 0.000 0.01" rpy="0 0 0"/>
+        </xacro:support_ce_module>
+      </xacro:if>
+      <!-- support_ce4: link4 -->
+      <xacro:if value="${self == 4}">
+        <xacro:support_ce_module name="support_ce4" parent="link4">
+          <origin xyz="${end_leg_offset} 0.000 0.01" rpy="0 0 0"/>
+        </xacro:support_ce_module>
+      </xacro:if>
+    </xacro:if>
     <!-- leg -->
     <xacro:if value="${with_leg == 1}">
@@ -270,9 +308,29 @@
         </xacro:standard_leg_old_version>
         </xacro:if>
-        <xacro:unless value="${old_version == 1}">
+        <!-- <xacro:unless value="${old_version == 1}">
           <xacro:standard_leg_joint parent = "link${self}" >
             <origin xyz="0.0 0.0 0" rpy="0 0 0"/>
           </xacro:standard_leg_joint>
-        </xacro:unless>
+        </xacro:unless> -->
+        <xacro:unless value="${old_version == 1}">
+        <!-- leg2: link2 に付ける -->
+        <xacro:if value="${self == 2}">
+          <xacro:standard_leg_joint parent="link2">
+            <origin xyz="0.05 0.0 0.01" rpy="0 0 0"/>
+          </xacro:standard_leg_joint>
+        </xacro:if>
+        <!-- leg3: link3 に付ける -->
+        <xacro:if value="${self == 3}">
+          <xacro:standard_leg_joint parent="link3">
+            <origin xyz="0.04 0.0 0.01" rpy="0 0 0"/>
+          </xacro:standard_leg_joint>
+        </xacro:if>
+        <!-- leg4: link4 ではなく link3 に付ける -->
+        <xacro:if value="${self == 4}">
+          <xacro:standard_leg_joint parent="link3">
+            <origin xyz="${link_length_3-0.05} 0.0 0.01" rpy="0 0 0"/>
+          </xacro:standard_leg_joint>
+        </xacro:if>
+      </xacro:unless>
         <!-- tail -->
         <xacro:if value="${self == links}">
@@ -296,5 +354,17 @@
         <parent link="link${self}"/>
         <child link="link${self+1}"/>
-        <origin rpy="0 0 0" xyz="${link_length} 0 0"/>
+        <!-- <origin rpy="0 0 0" xyz="${link_length} 0 0"/> -->
+        <xacro:if value="${self == 1}">
+        <!-- joint1: link1 -> link2 link_length = 0.6 -->
+          <origin rpy="0 0 0" xyz="${link_length} 0.000 0.000"/>
+        </xacro:if>
+        <xacro:if value="${self == 2}">
+          <!-- joint2: link2 -> link3 link_length = 0.575 -->
+          <origin rpy="0 0 0" xyz="${link_length_2} 0.000 0.000"/>
+        </xacro:if>
+        <xacro:if value="${self == 3}">
+          <!-- joint3: link3 -> link4 を調整 -->
+          <origin rpy="0 0 0" xyz="${link_length_3} 0.000 0.000"/>
+        </xacro:if>
         <axis xyz="0 0 1"/>
         <dynamics damping="0.9" friction="0.05"/>
