Commit message: [gimbalrotor][grape_with_arm] make the arm follow trajectories in gazebo
Derive joint5 gains from its 6.4e-8 kg m^2 inertia (the old ones diverged), raise joint4 i to cancel gravity, and drive the gripper mimic joints.
Set a 0.05 rad goal tolerance so an unreached goal is reported as GOAL_TOLERANCE_VIOLATED instead of succeeding.

File: robots/gimbalrotor/robots/grape_with_arm/gimbalrotor.gazebo.xacro (robot description, xacro)
@@ -15,3 +15,9 @@
   <xacro:joint_transmission joint="gimbal3"/>
   <xacro:joint_transmission joint="gimbal4"/>
+  <!-- the gripper joints follow arm_joint5_joint1 through <mimic>, which gazebo classic ignores -->
+  <gazebo>
+    <plugin name="mimic_joint_plugin" filename="libaerial_robot_mimic_joint_plugin.so">
+      <robotNamespace>$(arg robot_name)</robotNamespace>
+    </plugin>
+  </gazebo>
 </robot>
