Commit message: [gimbalrotor][grape_with_arm] put the centroid of the arm pipe on the pipe
screw_200mmpipe_module had its inertial in the frame of the CAD export: the centroid 1 m out along
the pipe (0.03, 0.02, 1.0), which is 0.221 m long, and the long axis of the inertia on x instead of z.
It put the model centroid of grape_with_arm 1.7 cm too far toward the arm (12.7 instead of 11.0 cm
ahead of the rotors in the pose of the flight of 2026-09-17), so the thrust was allocated for a robot
heavier on the arm side than the real one, which flew with the arm side up by 12-17 deg. The
centroid is now the middle of the pipe mesh (0, 0, 0.1105) and the inertia has its long axis on z; no
other link has its centroid outside its mesh. In gazebo the robot hovers level (roll and pitch within
0.1 deg).

File: robots/gimbalrotor/urdf/grape_with_arm/xacro/screw_200mmpipe_module.xacro (robot description, xacro)
@@ -9,8 +9,10 @@
     <link name="${prefix}base_link">
       <inertial>
-        <origin xyz="0.0314472120441254 0.0185600648406693 0.999996863971173" rpy="0.0 -0.0 0.0"/>
+        <!-- the pipe runs along z from the base (0) to the next module (0.221): the centroid and the
+             inertia were in the frame of the CAD export (1 m away, long axis on x), see the visual origin -->
+        <origin xyz="0.0 0.0 0.1105" rpy="0.0 0.0 0.0"/>
         <!-- <mass value="0.0784"/> -->
 	<mass value="0.0807"/>
-        <inertia ixx="1.92067336342704e-05" ixy="4.86844738251007e-08" ixz="-3.58103918098541e-08" iyy="0.000556258110321859" iyz="-3.52324723813976e-10" izz="0.000556910936857427"/>
+        <inertia ixx="0.000556910936857427" ixy="0.0" ixz="0.0" iyy="0.000556258110321859" iyz="0.0" izz="1.92067336342704e-05"/>
       </inertial>
       <visual>
