Commit message: Update grape drone model

File: robots/gimbalrotor/urdf/grape_with_arm/gimbalrotor.urdf.xacro (robot description, xacro)
@@ -69,7 +69,6 @@
     <visual>
       <geometry>
-        <mesh filename="package://gimbalrotor/urdf/grape/meshes/main_body.stl"/>
-      </geometry>
-      <material name="__unnamed_material_1"/>
+        <mesh filename="package://gimbalrotor/urdf/grape_with_arm/meshes/main_body.dae"/>
+      </geometry>
       <origin xyz="0.0 0.0 0.0" rpy="0.0 -0.0 0.0"/>
     </visual>
@@ -92,7 +91,6 @@
     <visual>
       <geometry>
-        <mesh filename="package://gimbalrotor/urdf/grape/meshes/gimbal1_link.stl"/>
-      </geometry>
-      <material name="__unnamed_material_2"/>
+        <mesh filename="package://gimbalrotor/urdf/grape_with_arm/meshes/gimbal1_link.dae"/>
+      </geometry>
       <origin xyz="0.0 0.0 0.0" rpy="0.0 -0.0 0.0"/>
     </visual>
@@ -107,7 +105,6 @@
     <visual>
       <geometry>
-        <mesh filename="package://gimbalrotor/urdf/grape/meshes/thrust1.stl"/>
-      </geometry>
-      <material name="__unnamed_material_3"/>
+        <mesh filename="package://gimbalrotor/urdf/grape_with_arm/meshes/thrust1.dae"/>
+      </geometry>
       <origin xyz="0.0 0.0 0.0" rpy="0.0 -0.0 0.0"/>
     </visual>
@@ -122,7 +119,6 @@
     <visual>
       <geometry>
-        <mesh filename="package://gimbalrotor/urdf/grape/meshes/gimbal2_link.stl"/>
-      </geometry>
-      <material name="__unnamed_material_4"/>
+        <mesh filename="package://gimbalrotor/urdf/grape_with_arm/meshes/gimbal2_link.dae"/>
+      </geometry>
       <origin xyz="0.0 0.0 0.0" rpy="0.0 -0.0 0.0"/>
     </visual>
@@ -137,7 +133,6 @@
     <visual>
       <geometry>
-        <mesh filename="package://gimbalrotor/urdf/grape/meshes/thrust2.stl"/>
-      </geometry>
-      <material name="__unnamed_material_5"/>
+        <mesh filename="package://gimbalrotor/urdf/grape_with_arm/meshes/thrust2.dae"/>
+      </geometry>
       <origin xyz="0.0 0.0 0.0" rpy="0.0 -0.0 0.0"/>
     </visual>
@@ -152,7 +147,6 @@
     <visual>
       <geometry>
-        <mesh filename="package://gimbalrotor/urdf/grape/meshes/gimbal3_link.stl"/>
-      </geometry>
-      <material name="__unnamed_material_6"/>
+        <mesh filename="package://gimbalrotor/urdf/grape_with_arm/meshes/gimbal3_link.dae"/>
+      </geometry>
       <origin xyz="0.0 0.0 0.0" rpy="0.0 -0.0 0.0"/>
     </visual>
@@ -167,7 +161,6 @@
     <visual>
       <geometry>
-        <mesh filename="package://gimbalrotor/urdf/grape/meshes/thrust3.stl"/>
-      </geometry>
-      <material name="__unnamed_material_7"/>
+        <mesh filename="package://gimbalrotor/urdf/grape_with_arm/meshes/thrust3.dae"/>
+      </geometry>
       <origin xyz="0.0 0.0 0.0" rpy="0.0 -0.0 0.0"/>
     </visual>
@@ -182,7 +175,6 @@
     <visual>
       <geometry>
-        <mesh filename="package://gimbalrotor/urdf/grape/meshes/gimbal4_link.stl"/>
-      </geometry>
-      <material name="__unnamed_material_8"/>
+        <mesh filename="package://gimbalrotor/urdf/grape_with_arm/meshes/gimbal4_link.dae"/>
+      </geometry>
       <origin xyz="0.0 0.0 0.0" rpy="0.0 -0.0 0.0"/>
     </visual>
@@ -197,7 +189,6 @@
     <visual>
       <geometry>
-        <mesh filename="package://gimbalrotor/urdf/grape/meshes/thrust4.stl"/>
-      </geometry>
-      <material name="__unnamed_material_9"/>
+        <mesh filename="package://gimbalrotor/urdf/grape_with_arm/meshes/thrust4.dae"/>
+      </geometry>
       <origin xyz="0.0 0.0 0.0" rpy="0.0 -0.0 0.0"/>
     </visual>

Commit message: [gimbalrotor][grape_with_arm] stand on the landing legs in gazebo
The only collision was a thin box at the body origin, so the legs sank 0.30 m into the ground.
Add collisions for the four foot pads and spawn grape_with_arm at z = 0.33 so the feet do not start inside the ground.

File: robots/gimbalrotor/urdf/grape_with_arm/gimbalrotor.urdf.xacro (robot description, xacro)
@@ -81,4 +81,21 @@
       <origin xyz="0.0 0.0 0.0" rpy="0.0 -0.0 0.0"/>
     </collision>
+    <!-- landing feet: pads at the bottom of the four legs of main_body.dae -->
+    <xacro:property name="foot_size" value="0.032 0.072 0.028"/>
+    <xacro:property name="foot_x" value="0.177"/>
+    <xacro:property name="foot_y" value="0.200"/>
+    <xacro:property name="foot_z" value="-0.304"/>
+    <xacro:macro name="foot_collision" params="sx sy">
+      <collision>
+        <geometry>
+          <box size="${foot_size}"/>
+        </geometry>
+        <origin xyz="${sx * foot_x} ${sy * foot_y} ${foot_z}" rpy="0.0 0.0 0.0"/>
+      </collision>
+    </xacro:macro>
+    <xacro:foot_collision sx="1" sy="1"/>
+    <xacro:foot_collision sx="1" sy="-1"/>
+    <xacro:foot_collision sx="-1" sy="1"/>
+    <xacro:foot_collision sx="-1" sy="-1"/>
   </link>
   <link name="gimbal1_link">

Commit message: [gimbalrotor][grape_with_arm] add RealSense D435 frames
Place camera_link and the depth/infra/color frames from the CAD, where the
front glass face of the D435 case sits at 0.118438 0 0.056 in main_body.
Offsets follow realsense2_description so the frames match the real camera.

File: robots/gimbalrotor/urdf/grape_with_arm/gimbalrotor.urdf.xacro (robot description, xacro)
@@ -426,4 +426,44 @@
   <!--   <origin xyz="0 0 -0.08" rpy="3.14159 0 0"/> -->
   <!-- </joint> -->
+  <!-- Intel RealSense D435.
+       The camera pose comes from dragons_quadrotor_module_witharm.SLDASM: the
+       centre of the front (glass) face of the case is at xyz="0.118438 0 0.056"
+       in main_body, looking straight along +x, upright, not tilted.
+       The frame layout and every offset below are realsense2_description's
+       urdf/_d435.urdf.xacro (ros2-development), so these frames match what
+       realsense2_camera publishes on the real robot:
+       https://github.com/IntelRealSense/realsense-ros/blob/ros2-development/realsense2_description/urdf/_d435.urdf.xacro
+       camera_link is the depth (left IR) frame: 4.3 mm behind the front glass
+       (zero-depth plane) and 17.5 mm to the left of the case centre. -->
+  <link name="camera_bottom_screw_frame"/>
+  <joint name="camera_joint" type="fixed">
+    <parent link="main_body"/>
+    <child link="camera_bottom_screw_frame"/>
+    <origin xyz="0.103538 0 0.0435" rpy="0 0 0"/>
+  </joint>
+  <link name="camera_link"/>
+  <joint name="camera_link_joint" type="fixed">
+    <parent link="camera_bottom_screw_frame"/>
+    <child link="camera_link"/>
+    <origin xyz="0.0106 0.0175 0.0125" rpy="0 0 0"/>
+  </joint>
+  <xacro:macro name="d435_sensor_frame" params="name y">
+    <link name="camera_${name}_frame"/>
+    <joint name="camera_${name}_joint" type="fixed">
+      <parent link="camera_link"/>
+      <child link="camera_${name}_frame"/>
+      <origin xyz="0 ${y} 0" rpy="0 0 0"/>
+    </joint>
+    <link name="camera_${name}_optical_frame"/>
+    <joint name="camera_${name}_optical_joint" type="fixed">
+      <parent link="camera_${name}_frame"/>
+      <child link="camera_${name}_optical_frame"/>
+      <origin xyz="0 0 0" rpy="${-pi/2} 0 ${-pi/2}"/>
+    </joint>
+  </xacro:macro>
+  <xacro:d435_sensor_frame name="depth"  y="0"/>
+  <xacro:d435_sensor_frame name="infra1" y="0"/>
+  <xacro:d435_sensor_frame name="infra2" y="-0.050"/>
+  <xacro:d435_sensor_frame name="color"  y="0.015"/>
   <!-- Include the arm macro -->
   <xacro:arm parent_link="main_body"/>

Commit message: [gimbalrotor][grape_with_arm] arm_pipe:=false for flying with the arm cut after the 90deg module

File: robots/gimbalrotor/urdf/grape_with_arm/gimbalrotor.urdf.xacro (robot description, xacro)
@@ -467,4 +467,6 @@
   <xacro:d435_sensor_frame name="color"  y="0.015"/>
   <!-- Include the arm macro -->
-  <xacro:arm parent_link="main_body"/>
+  <!-- arm_pipe:=false: the arm without the 200mm pipe and what follows it (joint1 and the 90deg module only) -->
+  <xacro:arg name="arm_pipe" default="true"/>
+  <xacro:arm parent_link="main_body" with_pipe="$(arg arm_pipe)"/>
 </robot>

File: robots/gimbalrotor/urdf/grape_with_arm/xacro/arm.xacro (robot description, xacro)
@@ -7,5 +7,7 @@
   <xacro:include filename="$(find gimbalrotor)/urdf/grape_with_arm/xacro/screw_drive_module_dynamixel.xacro"/>
   <xacro:include filename="$(find gimbalrotor)/urdf/grape_with_arm/xacro/vial_pick_module.xacro"/>
-  <xacro:macro name="arm" params="parent_link:=main_body xyz:='0.0995 0.0 -0.0465' rpy:='3.141592653589793 1.5707926535897934 3.141592653589793'">
+  <!-- with_pipe: false for the arm cut after the 90deg module (the 200mm pipe and all that follows it
+       taken off the real robot), so that the model keeps only joint1 and the 90deg module -->
+  <xacro:macro name="arm" params="parent_link:=main_body xyz:='0.0995 0.0 -0.0465' rpy:='3.141592653589793 1.5707926535897934 3.141592653589793' with_pipe:=true">
     <!-- Dummy link to attach the arm to the main body -->
     <link name="arm_dummy_link"/>
@@ -27,4 +29,5 @@
       xyz="0 0 0"
       rpy="0 3.14 -3.14159"/>
+    <xacro:if value="${with_pipe}">
     <!-- 200mm pipe module -->
     <xacro:screw_200mmpipe_module
@@ -69,4 +72,5 @@
       xyz="0 0 0"
       rpy="0 0 0"/>
+    </xacro:if>
     <!-- Transmissions for arm joints (required for Gazebo control) -->
     <transmission name="arm_joint1_tran">
@@ -80,4 +84,5 @@
       </actuator>
     </transmission>
+    <xacro:if value="${with_pipe}">
     <transmission name="arm_joint2_tran">
       <type>transmission_interface/SimpleTransmission</type>
@@ -120,4 +125,5 @@
       </actuator>
     </transmission>
+    </xacro:if>
   </xacro:macro>
 </robot>

Commit message: [gimbalrotor][grape_with_arm] move the body centroid back by the centroid measured in flight
The motor outputs of a flight without the arm pipe (2026-09-17 21:37, estimate_cog_from_flight.py)
put the centroid of the robot 8.3 mm behind the model (x 1.03 against 1.85 cm), and the robot flew
arm side up by 6-15 deg, as all the flights with the arm did. The centroid of main_body moves by
8.3 mm * 3.395 kg / 1.865 kg, to x 0.0027. Gazebo hovers level with and without the pipe.

File: robots/gimbalrotor/urdf/grape_with_arm/gimbalrotor.urdf.xacro (robot description, xacro)
@@ -54,5 +54,8 @@
     <inertial>
       <!-- <origin xyz="-0.0041019 0.0000721 -0.0183334" rpy="0.0 -0.0 0.0"/> -->
-      <origin xyz="0.0178508 0.0018366 -0.03525" rpy="0.0 -0.0 0.0"/>
+      <!-- x was 0.0178508 (CAD): the motor outputs of a hover without the arm pipe (2026-09-17 21:37, script/
+           estimate_cog_from_flight.py) put the centroid of the robot 8.3 mm behind the model, which flew arm
+           side up by 6-15 deg; the body centroid is moved by 8.3 mm * 3.395 kg / 1.865 kg -->
+      <origin xyz="0.0027468 0.0018366 -0.03525" rpy="0.0 -0.0 0.0"/>
       <!-- <mass value="1.3193189"/> -->
       <!-- <mass value="2.0421872">/ -->

Commit message: [gimbalrotor][grape_with_arm] weigh the body as the robot weighs
The robot without the arm pipe weighs 3.9 kg, 0.505 kg more than its model (3.395 kg), and climbed
slowly in its takeoffs while the z I control made up the thrust. The missing mass goes to main_body at
the centroid of the robot, so the centroid measured in flight stays, and the body inertia is scaled with
its mass. Gazebo hovers level with and without the pipe (3.9 and 4.635 kg).

File: robots/gimbalrotor/urdf/grape_with_arm/gimbalrotor.urdf.xacro (robot description, xacro)
@@ -54,19 +54,23 @@
     <inertial>
       <!-- <origin xyz="-0.0041019 0.0000721 -0.0183334" rpy="0.0 -0.0 0.0"/> -->
-      <!-- x was 0.0178508 (CAD): the motor outputs of a hover without the arm pipe (2026-09-17 21:37, script/
-           estimate_cog_from_flight.py) put the centroid of the robot 8.3 mm behind the model, which flew arm
-           side up by 6-15 deg; the body centroid is moved by 8.3 mm * 3.395 kg / 1.865 kg -->
-      <origin xyz="0.0027468 0.0018366 -0.03525" rpy="0.0 -0.0 0.0"/>
+      <!-- CAD: x 0.0178508, mass 1.8654999, inertia ixx 0.0233589 ixy -0.0000147 ixz -0.0001721 iyy 0.0237556
+           iyz -0.0000158 izz 0.0189000. Measured on 2026-09-17 without the arm pipe:
+           - the motor outputs of a hover (21:37, script/estimate_cog_from_flight.py) put the centroid of the
+             robot 8.3 mm behind the model, which flew arm side up by 6-15 deg: the body centroid was moved
+             by 8.3 mm * 3.395 kg / 1.865 kg to x 0.0027468
+           - the robot weighs 3.9 kg against 3.395 kg of the model: the missing 0.505 kg is added to the body at
+             the centroid of the robot (so the centroid stays), and the inertia is scaled with the mass -->
+      <origin xyz="0.0042073 0.0016796 -0.0314033" rpy="0.0 -0.0 0.0"/>
       <!-- <mass value="1.3193189"/> -->
       <!-- <mass value="2.0421872">/ -->
-      <mass value="1.8654999"/>
+      <mass value="2.3707399"/>
       <!-- <inertia ixx="0.0150906" ixy="-0.0000095" ixz="-0.0001112" iyy="0.0153469" iyz="-0.0000102" izz="0.0122100"/> -->
       <inertia
-	  ixx="0.0233589"
-	  ixy="-0.0000147"
-	  ixz="-0.0001721"
-	  iyy="0.0237556"
-	  iyz="-0.0000158"
-	  izz="0.0189000"/>
+	  ixx="0.0296853"
+	  ixy="-0.0000187"
+	  ixz="-0.0002187"
+	  iyy="0.0301894"
+	  iyz="-0.0000201"
+	  izz="0.0240188"/>
     </inertial>
     <visual>

Commit message: [gimbalrotor][grape_with_arm] move the body centroid by the centroid of the 22:15 hover
The motor outputs of the hover of 2026-09-17 22:15 (32 s, with the model at 3.9 kg) put the centroid
of the robot 2.5 mm behind and 2.3 mm left of the model, and the robot hovered left side down by 4 deg.
The body centroid moves by those times 3.9 kg / 2.371 kg. Gazebo hovers level with and without the pipe.

File: robots/gimbalrotor/urdf/grape_with_arm/gimbalrotor.urdf.xacro (robot description, xacro)
@@ -60,6 +60,9 @@
              by 8.3 mm * 3.395 kg / 1.865 kg to x 0.0027468
            - the robot weighs 3.9 kg against 3.395 kg of the model: the missing 0.505 kg is added to the body at
-             the centroid of the robot (so the centroid stays), and the inertia is scaled with the mass -->
-      <origin xyz="0.0042073 0.0016796 -0.0314033" rpy="0.0 -0.0 0.0"/>
+             the centroid of the robot (so the centroid stays), and the inertia is scaled with the mass
+           - a hover with that (22:15) put the centroid of the robot 2.5 mm behind and 2.3 mm left of the
+             model, and the robot hovered left side down by 4 deg: the body centroid moved from
+             (0.0042073, 0.0016796) by those times 3.9 kg / 2.371 kg -->
+      <origin xyz="0.0000947 0.0054632 -0.0314033" rpy="0.0 -0.0 0.0"/>
       <!-- <mass value="1.3193189"/> -->
       <!-- <mass value="2.0421872">/ -->
